File: Hardware/Electrodes input.kicad_sch (KiCad schematic)
At the start: 36 parts, among them J2 Conn_01x26_Pin, U10 TPD4E1B06DCKR, U2 TPD4E1B06DCKR, U3 TPD4E1B06DCKR, U4 TPD4E1B06DCKR, U5 TPD4E1B06DCKR, U9 TPD4E1B06DCKR

Commit message: Add Daisychain jumper
Parts:
- RN1, RN2, RN3, RN4: value 4.99 KΩ -> EXB-V8V512JV
Changed lines of the file:
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@@
 		(on_board yes)
 		(dnp no)
-		(fields_autoplaced yes)
 		(property "Reference" "C12"
 			(at 252.73 149.8537 0)
@@
 			)
 		)
-		(property "Value" "4.99 KΩ"
+		(property "Value" "EXB-V8V512JV"
 			(at 243.84 22.86 90)
 			(effects
@@
 		(on_board yes)
 		(dnp no)
-		(fields_autoplaced yes)
 		(property "Reference" "C36"
 			(at 260.35 149.8537 0)
@@
 			)
 		)
-		(property "Value" "4.99 KΩ"
+		(property "Value" "EXB-V8V512JV"
 			(at 243.84 130.81 90)
 			(effects
@@
 			)
 		)
-		(property "Value" "4.99 KΩ"
+		(property "Value" "EXB-V8V512JV"
 			(at 245.11 64.77 90)
 			(effects
@@
 		(on_board yes)
 		(dnp no)
-		(fields_autoplaced yes)
 		(property "Reference" "C26"
 			(at 256.54 149.8537 0)
@@
 			)
 		)
-		(property "Value" "4.99 KΩ"
+		(property "Value" "EXB-V8V512JV"
 			(at 245.11 99.06 90)
 			(effects

Commit message: TODO: GND pours & planes separation
Connections:
- net AGND: no longer J2.23 (Pin_23), J2.24 (Pin_24)
- net GNDA: now also J2.23 (Pin_23), J2.24 (Pin_24)
- net AVDD_ED renamed AVDD
Other:
- moved on the sheet: C11, C26, C36
