File: Hardware/bioamplifier.kicad_sch (KiCad schematic)
At the start: 45 parts, among them J1 Conn_01x07_Socket, J3 Conn_01x07_Socket, J4 Jumper, J5 Jumper, U1 ADS1299IPAG

Commit message: Add final changes
Parts:
- C5: footprint Capacitor_SMD:C_0603_1608Metric -> Capacitor_SMD:C_0805_2012Metric
Changed lines of the file:
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@@
 			)
 		)
-		(property "Footprint" "Capacitor_SMD:C_0603_1608Metric"
+		(property "Footprint" "Capacitor_SMD:C_0805_2012Metric"
 			(at 78.74 121.92 0)
 			(effects

Commit message: feat: add preview images
Parts:
- J4: footprint Connector_PinHeader_2.00mm:PinHeader_1x02_P2.00mm_Vertical -> Connector_PinHeader_2.54mm:PinHeader_1x02_P2.54mm_Vertical
Changed lines of the file:
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@@
 			)
 		)
-		(property "Footprint" "Connector_PinHeader_2.00mm:PinHeader_1x02_P2.00mm_Vertical"
+		(property "Footprint" "Connector_PinHeader_2.54mm:PinHeader_1x02_P2.54mm_Vertical"
 			(at 193.04 58.42 0)
 			(effects
